Commit message: tool0 should not be empty, otherwise collision checking will ignore end-effector

File: kuka_kr60_support/urdf/kr60ha.urdf (robot description, URDF)
Before this commit: robot kuka_kr60ha, 9 links, 8 joints
Links:
- link tool0: geometry collision sphere radius=0.001

File: kuka_kr60_support/urdf/kr60ha_macro.xacro (robot description, xacro)
@@ -159,5 +159,12 @@
     <!-- tool 0 -->
     <!-- This frame corresponds to the $FLANGE coordinate system in KUKA KRC controllers. -->
-    <link name="${prefix}tool0"/>
+    <link name="${prefix}tool0">
+      <collision>
+	<origin xyz="0 0 0" rpy="0 0 0"/>
+	<geometry>
+	  <sphere radius="0.001"/>
+	</geometry>
+      </collision>
+    </link>
     <!-- END LINKS -->
     <!-- JOINTS -->
