Commit message: Added cable guides etc to visual and collision model

File: kuka_kr60_support/urdf/kr60ha_macro.xacro (robot description, xacro)
@@ -84,5 +84,5 @@
         <origin xyz="0 0 0" rpy="0 0 0"/>
         <geometry>
-          <mesh filename="package://kuka_kr60_support/meshes/kr60ha/visual/link_3.dae" />
+          <mesh filename="package://kuka_kr60_support/meshes/kr60ha/visual/link_3.stl" />
         </geometry>
       </visual>
